File: Blackstone/Blackstone.kicad_sch (KiCad schematic)
At the start: 1 part, among them U1 STM32WL5MOCH6STR

Commit message: Create sheets
Parts:
- removed U1: STM32WL5MOCH6STR, LGA-92_10X10_STM, symbol STM32WL5MOC:STM32WL5MOCH6STR
- added J1: Conn_01x02_Pin, symbol Connector:Conn_01x02_Pin
- added J2: Conn_01x08_Socket, symbol Connector:Conn_01x08_Socket
- added J3: TC2030, Connector:Tag-Connect_TC2030-IDC-FP_2x03_P1.27mm_Vertical, symbol Connector:Conn_ARM_SWD_TagConnect_TC2030
- added J4: Conn_01x05_Pin, symbol Connector:Conn_01x05_Pin
- added P1: USB_C_Plug_USB2.0, symbol Connector:USB_C_Plug_USB2.0
Connections:
- new net +3V3: J3.1 (VCC), J4.3 (Pin_3)
- new net GND: J1.2 (Pin_2), J3.5 (GND), J4.5 (Pin_5), P1.A1 (GND), P1.A12 (GND), P1.B1 (GND), P1.B12 (GND), P1.S1 (SHIELD)
- new net Microcontroller/SWCLK: J3.4 (SWCLK), J4.1 (Pin_1)
- new net Microcontroller/SWDIO: J3.2 (SWDIO), J4.2 (Pin_2)
- new net Microcontroller/~{RESET}: J3.3 (~{RESET}), J4.4 (Pin_4)
- new net PYRO_MATCH,0-: J2.2 (Pin_2)
- new net PYRO_MATCH.0+: J2.1 (Pin_1)
- new net PYRO_MATCH.1+: J2.3 (Pin_3)
- new net PYRO_MATCH.1-: J2.4 (Pin_4)
- new net PYRO_MATCH.2+: J2.5 (Pin_5)
- new net PYRO_MATCH.2-: J2.6 (Pin_6)
- new net PYRO_MATCH.3+: J2.7 (Pin_7)
- new net PYRO_MATCH.3-: J2.8 (Pin_8)
- new net Power Supply/V_{BATT}: J1.1 (Pin_1)
- new net Power Supply/V_{USB}: P1.A4 (VBUS), P1.A9 (VBUS), P1.B4 (VBUS), P1.B9 (VBUS)
- new net USB.D+: P1.A6 (D+)
- new net USB.D-: P1.A7 (D-)
- no-connect marks 0 -> 1
Other:
- added sheet Accelerometer (accelerometer.kicad_sch)
- added sheet Altimeter (altimeter.kicad_sch)
- added sheet Data Logging Flash (flash.kicad_sch)
- added sheet GPS Module (gps.kicad_sch)
- added sheet IMU (imu.kicad_sch)
- added sheet Magnetometer (magnetometer.kicad_sch)
- added sheet Microcontroller (microcontroller.kicad_sch)
- added sheet Power Supply (power_supply.kicad_sch)
- added sheet Pyros (pryos.kicad_sch)
- added sheet USB to Serial (usb_serial.kicad_sch)
- note added: "Battery Connector"
- note added: "SWD Connectors"
- title: Blackstone Flight Computer -> Blackstone Flight Computer - Overview
