File: Blackstone/flash.kicad_sch (KiCad schematic)
At the start: 0 parts

Commit message: Set sheet titles
Other:
- title: Blackstone Flight Computer - Overview -> Blackstone Flight Computer - Data Logging Flash
Changed lines of the file:
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@@
 	(paper "A4")
 	(title_block
-		(title "Blackstone Flight Computer - Overview")
+		(title "Blackstone Flight Computer - Data Logging Flash")
 		(date "2024-08-02")
 		(rev "Rev A")
