File: Blackstone/microcontroller.kicad_sch (KiCad schematic)
At the start: 1 part, among them U1 STM32WL55CCUx

Commit message: Set sheet titles
Other:
- title: Blackstone Flight Computer - Overview -> Blackstone Flight Computer - Microcontroller
Changed lines of the file:
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@@
 	(paper "A4")
 	(title_block
-		(title "Blackstone Flight Computer - Overview")
+		(title "Blackstone Flight Computer - Microcontroller")
 		(date "2024-08-02")
 		(rev "Rev A")
@@
 	(label "GPS_UART.TX"
 		(at 162.56 64.77 0)
+		(fields_autoplaced yes)
 		(effects
 			(font
@@
 	(label "GPS_UART.RX"
 		(at 162.56 67.31 0)
+		(fields_autoplaced yes)
 		(effects
 			(font
