File: Blackstone/pryos.kicad_sch (KiCad schematic)
At the start: 0 parts

Commit message: Set sheet titles
Other:
- title: Blackstone Flight Computer - Overview -> Blackstone Flight Computer - Pyros
Changed lines of the file:
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@@
 	(paper "A4")
 	(title_block
-		(title "Blackstone Flight Computer - Overview")
+		(title "Blackstone Flight Computer - Pyros")
 		(date "2024-08-02")
 		(rev "Rev A")
